Commit message: fix: weird urdf

File: src/lerobot/model/uh-right/uh-right.urdf (robot description, URDF)
Before this commit: robot UH-v3.0 final.SLDASM right, 8 links, 7 joints
Links:
- link Link7: mass 0.0603672149333555 -> 0.0603671967995476
Joints:
- joint joint1: axis 0 0 -1 -> 0 0 1; origin xyz=-0.0038974 -0.073 -0.0125 rpy=1.5708 0 0 -> xyz=0.0038974 0.073 0.0125 rpy=-1.5708 0 0
- joint joint2: limit lower=0 upper=0 effort=0 velocity=0 -> lower=-3.14 upper=3.14 effort=0.5 velocity=100; origin xyz=-0.0173 0 0.068 rpy=-1.5708 0 1.5708 -> xyz=-0.0173 0 0.068 rpy=1.5708 0 -1.5708
- joint joint3: axis 0 0 -1 -> 0 0 1; limit lower=0 upper=0 effort=0 velocity=0 -> lower=-3.14 upper=3.14 effort=0.5 velocity=100; origin xyz=0.075 0 -0.0173 rpy=0 1.5708 0 -> xyz=-0.075 0 -0.0173 rpy=0 -1.5708 0
- joint joint4: limit lower=0 upper=0 effort=0 velocity=0 -> lower=-3.14 upper=3.14 effort=0.5 velocity=100; origin xyz=0.0173 0 0.128 rpy=0 1.5708 0 -> xyz=0.0173 0 0.128 rpy=0 -1.5708 0
- joint joint5: axis 0 0 -1 -> 0 0 1; limit lower=0 upper=0 effort=0 velocity=0 -> lower=-3.14 upper=3.14 effort=0.5 velocity=100; origin xyz=-0.065027 -0.0044352 -0.0173 rpy=0 -1.5708 0 -> xyz=0.065178 0 0.0173 rpy=0 1.5708 0
- joint joint6: limit lower=0 upper=0 effort=0 velocity=0 -> lower=-3.14 upper=3.14 effort=0.5 velocity=100; origin xyz=0.0173 0.0044352 0.077151 rpy=0 1.5708 0 -> xyz=-0.0173 0 0.077 rpy=0 -1.5708 0
- joint joint7: limit lower=0 upper=0 effort=0 velocity=0 -> lower=-3.14 upper=3.14 effort=0.5 velocity=100; origin xyz=-0.09 0 -0.0173 rpy=0 -1.5708 0 -> xyz=0.09 0 -0.0173 rpy=0 1.5708 0

File: src/lerobot/model/uh-right/urdf/UH-v3.0 final.SLDASM right v2.urdf (robot description, URDF)
Before this commit: robot UH-v3.0 final.SLDASM right, 8 links, 7 joints
Links:
- link Link1: geometry collision mesh filename=package://UH-v3.0 final.SLDASM right v2/meshes/Link1.STL; visual mesh filename=package://UH-v3.0 final.SLDASM right v2/meshes/Link1.STL
- link Link2: geometry collision mesh filename=package://UH-v3.0 final.SLDASM right v2/meshes/Link2.STL; visual mesh filename=package://UH-v3.0 final.SLDASM right v2/meshes/Link2.STL
- link Link3: geometry collision mesh filename=package://UH-v3.0 final.SLDASM right v2/meshes/Link3.STL; visual mesh filename=package://UH-v3.0 final.SLDASM right v2/meshes/Link3.STL
- link Link4: geometry collision mesh filename=package://UH-v3.0 final.SLDASM right v2/meshes/Link4.STL; visual mesh filename=package://UH-v3.0 final.SLDASM right v2/meshes/Link4.STL
- link Link5: geometry collision mesh filename=package://UH-v3.0 final.SLDASM right v2/meshes/Link5.STL; visual mesh filename=package://UH-v3.0 final.SLDASM right v2/meshes/Link5.STL
- link Link6: geometry collision mesh filename=package://UH-v3.0 final.SLDASM right v2/meshes/Link6.STL; visual mesh filename=package://UH-v3.0 final.SLDASM right v2/meshes/Link6.STL
- link Link7: mass 0.0603672149333555 -> 0.0603671967995476; geometry collision mesh filename=package://UH-v3.0 final.SLDASM right v2/meshes/Link7.STL; visual mesh filename=package://UH-v3.0 final.SLDASM right v2/meshes/Link7.STL
- link base_link: geometry collision mesh filename=package://UH-v3.0 final.SLDASM right v2/meshes/base_link.STL; visual mesh filename=package://UH-v3.0 final.SLDASM right v2/meshes/base_link.STL
Joints:
- joint joint1: axis 0 0 -1 -> 0 0 1; origin xyz=-0.0038974 -0.073 -0.0125 rpy=1.5708 0 0 -> xyz=0.0038974 0.073 0.0125 rpy=-1.5708 0 0
- joint joint2: origin xyz=-0.0173 0 0.068 rpy=-1.5708 0 1.5708 -> xyz=-0.0173 0 0.068 rpy=1.5708 0 -1.5708
- joint joint3: axis 0 0 -1 -> 0 0 1; origin xyz=0.075 0 -0.0173 rpy=0 1.5708 0 -> xyz=-0.075 0 -0.0173 rpy=0 -1.5708 0
- joint joint4: origin xyz=0.0173 0 0.128 rpy=0 1.5708 0 -> xyz=0.0173 0 0.128 rpy=0 -1.5708 0
- joint joint5: axis 0 0 -1 -> 0 0 1; origin xyz=-0.065027 -0.0044352 -0.0173 rpy=0 -1.5708 0 -> xyz=0.065178 0 0.0173 rpy=0 1.5708 0
- joint joint6: origin xyz=0.0173 0.0044352 0.077151 rpy=0 1.5708 0 -> xyz=-0.0173 0 0.077 rpy=0 -1.5708 0
- joint joint7: origin xyz=-0.09 0 -0.0173 rpy=0 -1.5708 0 -> xyz=0.09 0 -0.0173 rpy=0 1.5708 0
