Commit message: better calibrate

File: src/lerobot/model/uh/uh.urdf (robot description, URDF)
Before this commit: robot UH-v3.0 final.SLDASM v9, 8 links, 7 joints
Joints:
- joint joint1: axis 0 0 -1 -> 0 0 1
- joint joint2: axis 0 0 1 -> 0 0 -1
- joint joint4: axis 0 0 -1 -> 0 0 1
- joint joint5: axis 0 0 -1 -> 0 0 1
- joint joint6: axis 0 0 -1 -> 0 0 1
- joint joint7: axis 0 0 -1 -> 0 0 1
